Commit message: Implemented car like xml

File: carlike.urdf (robot description, URDF)
Before this commit: robot car_like_robot, 5 links, 4 joints
Links:
- removed link front_wheel
- removed link rear_wheel
- removed link steering_link
- added link front_left_steer
- added link front_left_wheel; visual cylinder length=0.05 radius=0.1
- added link front_right_steer
- added link front_right_wheel; visual cylinder length=0.05 radius=0.1
- added link rear_left_wheel; visual cylinder length=0.05 radius=0.1
- added link rear_right_wheel; visual cylinder length=0.05 radius=0.1
- link base_link: geometry collision box size=0.5 0.3 0.1; visual box size=0.5 0.2 0.1
Joints:
- removed joint front_wheel_joint
- removed joint rear_wheel_joint
- removed joint steering_joint
- added joint front_left_steer_joint: type revolute, parent base_link, child front_left_steer, origin xyz=0.20 0.15 -0.05, axis 0 0 1, limit lower=-0.6109 upper=0.6109 effort=10 velocity=1
- added joint front_left_wheel_joint: type fixed, parent front_left_steer, child front_left_wheel, origin xyz=0 0 0
- added joint front_right_steer_joint: type revolute, parent base_link, child front_right_steer, origin xyz=0.20 -0.15 -0.05, axis 0 0 1, limit lower=-0.6109 upper=0.6109 effort=10 velocity=1
- added joint front_right_wheel_joint: type fixed, parent front_right_steer, child front_right_wheel, origin xyz=0 0 0
- added joint rear_left_wheel_joint: type fixed, parent base_link, child rear_left_wheel, origin xyz=-0.20 0.15 -0.05
- added joint rear_right_wheel_joint: type fixed, parent base_link, child rear_right_wheel, origin xyz=-0.20 -0.15 -0.05
